File: PCB Design/CuttleBoard_8Layers.kicad_sch (KiCad schematic)
At the start: 170 parts, among them IC1 W25Q256JVEIQ TR, J1 DX07WH24JA3R1200, SW1 SW_Push, U1 LMR33630CQRNX, U15 TPS62824ADMQ, U16 ICM-20602, U19 USBLC6-2P6, U2 STM32H735VGH6, U20 ACS722xLCTR-10AB, U3 LMR33630CQRNX, U4 ICM-20602, U7 MPRLS0025PA00001A, Y1 NX2016SA

Commit message: redone schematics for H743VIT
Parts:
- removed C21, C22, C23: 4.7µF, Capacitor_SMD:C_0402_1005Metric, symbol Device:C
- removed L3: 2.2µH, Inductor_SMD:L_0603_1608Metric, symbol pspice:INDUCTOR
- removed U2: STM32H735VGH6, Package_BGA:TFBGA-100_8x8mm_Layout10x10_P0.8mm, symbol ultimateFC-rescue:STM32H735VGH6-lib_ultimateFC
- added C14, C16: 4.7µF, Capacitor_SMD:C_0402_1005Metric, symbol Device:C
- added C19: 100nF, Capacitor_SMD:C_0402_1005Metric, symbol Device:C
- added SW2: SW_Push, Button_Switch_SMD:SW_Push_1P1T-SH_NO_CK_KMR2xxG, symbol Switch:SW_Push
- added U14: STM32H743VIHx, Package_BGA:TFBGA-100_8x8mm_Layout10x10_P0.8mm, symbol MCU_ST_STM32H7:STM32H743VIHx
- R20: value 2k2 -> 10k; footprint Resistor_SMD:R_0402_1005Metric -> ultimateFC:R_0201_0603Metric_mod; JLCPCB Part # C2076947 -> (none)
- R9: value 10k -> 2k2; footprint ultimateFC:R_0201_0603Metric_mod -> Resistor_SMD:R_0402_1005Metric; JLCPCB Part # (none) -> C2076947
Connections:
- net CS_FLASH: now also U14.C3 (PE4)
- net CS_IMU1: now also U14.C7 (PD3)
- net CS_IMU2: now also U14.C4 (PE1)
- net CS_IMU3: now also U14.D6 (PD7)
- net EOC_PRESSURE: now also U14.A2 (PC13)
- net GND: now also R9.2, C14.2, C16.2, C19.2, SW2.1, U14.C2 (VSS), U14.E4 (VSS), U14.E5 (VSS), U14.E6 (VSS), U14.G1 (VSSA), U14.J1 (VSS); no longer R20.2
- net I2C1_SCL: now also U14.B4 (PB8)
- net I2C1_SDA: now also U14.A4 (PB9)
- net I2C2_SCL: now also U14.J7 (PB10)
- net I2C2_SDA: now also U14.K7 (PB11)
- net I2C3_SCL: now also U14.D9 (PA8)
- net I2C3_SDA: now also U14.E9 (PC9)
- net I2C4_SCL: now also U14.B5 (PB6)
- net I2C4_SDA: now also U14.A5 (PB7)
- net INT_IMU1: now also U14.B7 (PD2)
- net INT_IMU2: now also U14.C5 (PB5)
- net NRST: now also R20.2, C19.1, SW2.2, U14.E1 (NRST); no longer R9.2
- net OSC_IN: now also C9.1, U14.C1 (PH0); no longer C7.1
- net OSC_OUT: now also C7.1, U14.D1 (PH1); no longer C9.1
- net RES_PRESSURE: now also U14.B3 (PE3)
- net SWDCLK: now also U14.A9 (PA14)
- net SWDIO: now also U14.A10 (PA13)
- net UART3_RX: now also U14.J9 (PD9)
- net UART3_TX: now also U14.K9 (PD8)
- net UART7_RX: now also U14.H5 (PE7)
- net USB_D+: now also U14.B10 (PA12)
- net USB_D-: now also U14.C10 (PA11)
- net VSense: now also U14.G4 (PC4)
- net curr_sig: now also U14.J3 (PA6)
- net +3.3V: now reaches R20.1
- net +3.3V: now also C20.1, C31.1, C32.1, C33.1, C34.1, C35.1, C36.1, C37.1, C38.1, C39.1, C40.1, C41.1, C42.1, C43.1, C44.1, C45.1, C46.1, C47.1, C49.1, FB7.1, IC1.8 (VCC), JP1.1 (A), R18.1, R19.1, R2.1, R21.1, R22.1, R23.1, R3.1, R7.1, R8.1, SW1.2, TP44.1, TP45.1, TP7.1, TP8.1, TP9.1, U16.1 (VDDIO), U16.16 (VDD), U17.5 (VDD_IO), U17.8 (VDD), U20.8 (VCC), U4.1 (VDDIO), U4.16 (VDD), U7.12 (VDD), U14.B2 (VBAT), U14.D2 (VDD), U14.F4 (VDDLDO), U14.F5 (VDD), U14.F6 (VDD33_USB), U14.F7 (PDR_ON), U14.H1 (VDDA), U14.K1 (VDD); no longer SW1.1
- removed net +3V3: C20.1, C31.1, C32.1, C33.1, C34.1, C35.1, C36.1, C37.1, C38.1, C39.1, C40.1, C41.1, C42.1, C43.1, C44.1, C45.1, C46.1, C47.1, C49.1, FB7.1, IC1.8 (VCC), JP1.1 (A), R18.1, R19.1, R2.1, R21.1, R22.1, R23.1, R3.1, R7.1, R8.1, R9.1, SW1.2, TP44.1, TP45.1, TP7.1, TP8.1, TP9.1, U16.1 (VDDIO), U16.16 (VDD), U17.5 (VDD_IO), U17.8 (VDD), U20.8 (VCC), U4.1 (VDDIO), U4.16 (VDD), U7.12 (VDD)
- net INT_IMU31 renamed INT1_IMU3
- net INT1_IMU3: now also U14.D7 (PD4)
- net INT_IMU32 renamed INT2_IMU3
- net INT2_IMU3: now also U14.D8 (PD0)
- net MISO_GYRO renamed SPI3_MISO
- net SPI3_MISO: now also U14.B8 (PC11)
- net MOSI_GYRO renamed SPI3_MOSI
- net SPI3_MOSI: now also U14.C8 (PC12)
- net PA9_USB_VBUS_sense: no longer names the net of R14.2, R15.1, TP81.1
- net PC7_LED_WT renamed LED_WT
- net LED_WT: now also U14.F9 (PC8)
- net PC8_LED_BL renamed LED_BL
- net LED_BL: now also U14.H9 (PD10)
- net SCLK_GYRO renamed SPI3_SCK
- net SPI3_SCK: now also U14.B9 (PC10)
- net UART4_RX renamed UART2_RX
- net UART2_RX: now also U14.C6 (PD6)
- net UART4_TX renamed UART2_TX
- net UART2_TX: now also U14.B6 (PD5)
- net UART9_RX renamed UART5_RX
- net UART5_RX: now also U14.K8 (PB12)
- net UART9_TX renamed UART5_TX
- net UART5_TX: now also U14.J8 (PB13)
- new net: C14.1, U14.E7 (VCAP)
- new net: C16.1, U14.F8 (VCAP)
- new net BOOT0: R9.1, SW1.1, U14.D5 (BOOT0)
Other:
- note removed: "Application Note (AN5419)"
- note removed: "MISO"
- note removed: "next to PD10 or PD11"
- moved on the sheet: C10, C11, C12, C13, C17, C18, C24, C28, C29, C3, C30, C31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

Commit message: good progress, needs checking, 14 violations to fix
Connections:
- net CS_IMU2: now also U14.A7 (PB3); no longer U14.C4 (PE1)
- net CS_IMU3: now also U14.A6 (PB4); no longer U14.D6 (PD7)
- net INT1_IMU3: now also U14.C4 (PE1); no longer U14.D7 (PD4)
- net INT2_IMU3: now also U14.C5 (PB5); no longer U14.D8 (PD0)
- net INT_IMU2: now also U14.A8 (PA15); no longer U14.C5 (PB5)
