File: PCB Design/Coil_Drivers.kicad_sch (KiCad schematic)
At the start: 8 parts

Commit message: Revert "STM32H743 first version"
Connections:
- net GND: no longer U10.16 (GND), U10.2 (GND), U10.5 (GND), U11.16 (GND), U11.2 (GND), U11.5 (GND), U12.16 (GND), U12.2 (GND), U12.5 (GND), U13.16 (GND), U13.2 (GND), U13.5 (GND)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
- no-connect marks 64 -> 16
